Commit message: hand-camera coordination complete with different camera positioning

File: cp25_webapp/Universal_Robots_ROS2_Description/urdf/ur.urdf.xacro (robot description, xacro)
@@ -94,4 +94,7 @@
        <!--<origin xyz="0.0 0 0.0" rpy="0 -1.57 1.57"/>-->
    </xacro:rg2_gripper>
+   <!--peerajak this is originalxacro:sensor_r430 prefix="wrist_rgbd" parent="base_link" >
+       <origin xyz="-0.25 -0.3 0.2" rpy="0 ${pi/3} ${pi/2}"/>
+   </xacro:sensor_r430 peerajak this is original-->
    <xacro:sensor_r430 prefix="wrist_rgbd" parent="base_link" >
        <origin xyz="-0.25 -0.3 0.2" rpy="0 ${pi/3} ${pi/2}"/>
